File: Hardware/ESP32 drone.kicad_pcb (KiCad board)
At the start: 2 copper layers, 100 x 100 mm, 131 parts, among them IC1 TP4056, J1 USB_C_Receptacle_USB2.0, J2 Conn_01x02_Female, J3 B2B-PH-SM4-TB(LF)(SN), J4 Conn_01x02_Female, J5 Conn_01x02_Female, J6 Conn_01x02_Female, J8 Conn_01x06_Female, J9 Conn_01x06_Female, SW1 K3-1280S-F1, T1 SI2302DS-T1, T2 SI2302DS-T1, T3 SI2302DS-T1, T4 SI2302DS-T1, U1 100K, U2 AO3401, U3 MIC5219-3.3YM5, U4 100K, U5 100K, U6 CP2102N-Axx-xQFN28, U7 2N7002DW, U8 ESP32-WROOM-32, U9 MPU-6050

Commit message: Organize drawings and BOM
Parts:
- removed REF** (x56): 1mm hole, ESP32_TouchDown_lib:1mm hole
- removed U1: 100K, Resistor_SMD:R_0603_1608Metric
- removed U2: AO3401, Package_TO_SOT_SMD:SOT-23
- added Q1: AO3401A, Package_TO_SOT_SMD:SOT-23, F.Cu at (145.3, 73.9)
- added R22: 100k, Resistor_SMD:R_0603_1608Metric, F.Cu at (144.1, 70.6)
- C1, C4: value 10u -> 10uF
- C12: value 0.1uf -> 0.1uF
- D2, D3, D4, D5: footprint Diode_SMD:D_SOD-323 -> Diode_SMD:D_SOD-123
- IC1: footprint tp4056:SOIC127P600X175-9N -> loc_footprints:SOIC127P600X175-9N
- J2, J4, J5, J6: value Conn_01x02_Female -> Conn_01x02_Socket
- J3: value B2B-PH-SM4-TB(LF)(SN) -> B2B-PH-SM4-TB(LF)(SN)
- J8, J9: value Conn_01x06_Female -> Conn_01x06_Socket
- R3, R4: value 1.3K -> 1k3
- SW1: value K3-1280S-F1 -> K3-1280S-F1; footprint ESP32_TouchDown_lib:slide switch spdt -> loc_footprints:slide switch spdt
- T1, T2, T3, T4: footprint SI2302DS-T1:SOT95P237X112-3N -> loc_footprints:SOT95P237X112-3N
- U7: value 2N7002DW -> DDC114TU-7-F
- U9: footprint MPU6050:MPU6050 -> loc_footprints:MPU6050
Connections:
- net /ADC_BAT renamed /MCU/ADC_BAT
- net /D+ renamed /Debug/D+
- net /D- renamed /Debug/D-
- net /DTR renamed /Debug/DTR
- net /EN renamed /Debug/EN
- net /EXI5 renamed /MCU/EXI5
- net /EXIO1 renamed /MCU/EXIO1
- net /EXIO2 renamed /MCU/EXIO2
- net /EXIO3 renamed /MCU/EXIO3
- net /EXIO4 renamed /MCU/EXIO4
- net /IO0 renamed /Debug/IO0
- net /LDO_H renamed /Power/LDO_H
- net /LED_1 renamed /Debug/LED1
- net /LED_2 renamed /Debug/LED2
- net /LED_3 renamed /Debug/LED3
- net /MOT_1 renamed /MCU/MOTOR1
- net /MOT_2 renamed /MCU/MOTOR2
- net /MOT_3 renamed /MCU/MOTOR3
- net /MOT_4 renamed /MCU/MOTOR4
- net /RTS renamed /Debug/RTS
- net /RX renamed /Debug/TXD
- net /RXD2 renamed /MCU/RXD2
- net /SCL renamed /MCU/SCL
- net /SDA renamed /MCU/SDA
- net /SRV_1 renamed /MCU/SRV_1
- net /SRV_2 renamed /MCU/SRV_2
- net /SRV_3 renamed /MCU/SRV_3
- net /SRV_4 renamed /MCU/SRV_4
- net /TX renamed /Debug/RXD
- net /TXD2 renamed /MCU/TXD2
